File: VanController.kicad_pcb (KiCad board)
At the start: 4 copper layers, 230 x 135 mm, 253 parts, among them J1 +12V IN (M5 stud), J10 NO / COM / NC, J11 LOAD+ / LOAD-, J12 LOAD+ / LOAD-, J13 LOAD+ / LOAD-, J14 LOAD+ / LOAD-, J15 LOAD+ / LOAD-, J16 LOAD+ / LOAD-, J17 CANH / CANL / GND, J18 A / B / GND, J19 GPS ANT (u.FL), J2 GND IN (M5 stud), J20 AUX ADC, J21 WATER 1, J22 WATER 2, J3 USB-C, J4 UART0 debug, J5 NO / COM / NC, J6 NO / COM / NC, J7 NO / COM / NC, J8 NO / COM / NC, J9 NO / COM / NC, K1 G5LE-1-E DC12, K2 G5LE-1-E DC12, K3 G5LE-1-E DC12, K4 G5LE-1-E DC12, K5 G5LE-1-E DC12, K6 G5LE-1-E DC12, Q1 CSD18540Q5B, Q10 BUK9M12-60EX, Q11 BUK9M12-60EX, Q12 BUK9M12-60EX, Q13 BUK9M12-60EX, Q14 BUK9M12-60EX, Q2 CSD18540Q5B, Q3 AO3400A, Q4 AO3400A, Q5 AO3400A, Q6 AO3400A, Q7 AO3400A, Q8 AO3400A, Q9 BUK9M12-60EX, SW1 RESET, SW2 BOOT, U1 LM74700QDBVRQ1, U10 ADS1115IDGS, U11 TCA9535PWR, U2 TPS54360DDA, U3 AMS1117-3.3, U4 ESP32-S3-WROOM-1-N16, U5 USBLC6-2SC6, U6 TJA1051T/3, U7 THVD1450D, U8 MAX-M10S, U9 LIS3DH

Commit message: Rev 0.3a: dry-contact option for the relay outputs
Each relay channel gets a bridged solder jumper (SJ1-SJ6) between the
fused COM copper and the fuse-sense resistor. Removing the channel fuse
and cutting the jumper leaves COM/NO/NC connected only to the relay
contacts. Copper-only change: Gerbers regenerated, BOM and centroid
unchanged. make_fab.py now writes UTC timestamps and zips the Gerbers.
Docs: dry-contact procedure, firmware note, PCBWay loose-parts note.

Co-Authored-By: Claude Opus 5.5 <noreply@anthropic.com>
Parts:
- added SJ1: DRY (cut), Jumper:SolderJumper-2_P1.3mm_Bridged_RoundedPad1.0x1.5mm, F.Cu at (59.3, 91.8)
- added SJ2: DRY (cut), Jumper:SolderJumper-2_P1.3mm_Bridged_RoundedPad1.0x1.5mm, F.Cu at (80.3, 91.8)
- added SJ3: DRY (cut), Jumper:SolderJumper-2_P1.3mm_Bridged_RoundedPad1.0x1.5mm, F.Cu at (101.3, 91.8)
- added SJ4: DRY (cut), Jumper:SolderJumper-2_P1.3mm_Bridged_RoundedPad1.0x1.5mm, F.Cu at (122.3, 91.8)
- added SJ5: DRY (cut), Jumper:SolderJumper-2_P1.3mm_Bridged_RoundedPad1.0x1.5mm, F.Cu at (143.3, 91.8)
- added SJ6: DRY (cut), Jumper:SolderJumper-2_P1.3mm_Bridged_RoundedPad1.0x1.5mm, F.Cu at (164.3, 91.8)
Connections:
- R33 pad 1: /Relays/Relay1/OUT_F -> /Relays/Relay1/SENSE_TAP
- R34 pad 1: /Relays/Relay2/OUT_F -> /Relays/Relay2/SENSE_TAP
- R35 pad 1: /Relays/Relay3/OUT_F -> /Relays/Relay3/SENSE_TAP
- R36 pad 1: /Relays/Relay4/OUT_F -> /Relays/Relay4/SENSE_TAP
- R37 pad 1: /Relays/Relay5/OUT_F -> /Relays/Relay5/SENSE_TAP
- R38 pad 1: /Relays/Relay6/OUT_F -> /Relays/Relay6/SENSE_TAP
Routing:
- net /Relays/Relay3/OUT_F: track 134.4 -> 106.0 mm, vias 1 -> 0
- net /Relays/Relay6/OUT_F: track 134.4 -> 106.0 mm, vias 1 -> 0
- net /Relays/Relay4/OUT_F: track 134.4 -> 106.0 mm, vias 1 -> 0
- net /Relays/Relay5/OUT_F: track 134.4 -> 106.0 mm, vias 1 -> 0
- net /Relays/Relay2/OUT_F: track 134.3 -> 106.0 mm, vias 1 -> 0
- net /Relays/Relay3/SENSE_TAP: track 0.00 -> 27.5 mm, vias 0 -> 2
- net /Relays/Relay6/SENSE_TAP: track 0.00 -> 27.5 mm, vias 0 -> 2
- net /Relays/Relay4/SENSE_TAP: track 0.00 -> 27.5 mm, vias 0 -> 2
- net /Relays/Relay5/SENSE_TAP: track 0.00 -> 27.5 mm, vias 0 -> 2
- net /Relays/Relay1/OUT_F: track 133.5 -> 106.0 mm, vias 1 -> 0
- net /Relays/Relay2/SENSE_TAP: track 0.00 -> 27.5 mm, vias 0 -> 2
- net /Relays/Relay1/SENSE_TAP: track 0.00 -> 26.6 mm, vias 0 -> 2
Other:
- board text added: "VanController rev 0.3a"
- board text removed: "VanController rev 0.3"
