File: relay_channel.kicad_sch (KiCad schematic)
At the start: 13 parts, among them J5 NO / COM / NC, K1 G5LE-1-E DC12, Q3 AO3400A

Commit message: Rev 0.3a: dry-contact option for the relay outputs
Each relay channel gets a bridged solder jumper (SJ1-SJ6) between the
fused COM copper and the fuse-sense resistor. Removing the channel fuse
and cutting the jumper leaves COM/NO/NC connected only to the relay
contacts. Copper-only change: Gerbers regenerated, BOM and centroid
unchanged. make_fab.py now writes UTC timestamps and zips the Gerbers.
Docs: dry-contact procedure, firmware note, PCBWay loose-parts note.

Co-Authored-By: Claude Opus 5.5 <noreply@anthropic.com>
Parts:
- added SJ1: DRY (cut), Jumper:SolderJumper-2_P1.3mm_Bridged_RoundedPad1.0x1.5mm, symbol Jumper:SolderJumper_2_Bridged
Connections:
- net OUT_F: now also SJ1.1 (A); no longer R33.1
- new net SENSE_TAP: R33.1, SJ1.2 (B)
Other:
- note added: "Relay channel. COM is fed from +12V through the channel fuse, so NO gives switched, fused +12 V. FUSE_SENSE is high (~2.8 V at 12 V) while the fuse is intact; BAT54S clamps transients to +3V3. DRY CONTACT: remove the fuse and cut solder jumper SJ (DRY). COM/NO/NC then connect only to the relay contacts; FUSE_SENSE reads low (firmware: treat as dry-contact mode). Not rated for mains."
- note removed: "Relay channel. COM is fed from +12V through the channel fuse, so NO gives switched, fused +12 V. FUSE_SENSE is high (~2.8 V at 12 V) while the fuse is intact; BAT54S clamps transients to +3V3."
Changed lines of the file:
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@@
 		(company "VanController")
 	)
-	(text "Relay channel. COM is fed from +12V through the channel fuse, so NO gives switched, fused +12 V. FUSE_SENSE is high (~2.8 V at 12 V) while the fuse is intact; BAT54S clamps transients to +3V3."
+	(text "Relay channel. COM is fed from +12V through the channel fuse, so NO gives switched, fused +12 V. FUSE_SENSE is high (~2.8 V at 12 V) while the fuse is intact; BAT54S clamps transients to +3V3. DRY CONTACT: remove the fuse and cut solder jumper SJ (DRY). COM/NO/NC then connect only to the relay contacts; FUSE_SENSE reads low (firmware: treat as dry-contact mode). Not rated for mains."
 		(exclude_from_sim no)
 		(at 20.32 15.24 0)
@@
 		)
 	)
-	(label "OUT_F"
+	(label "SENSE_TAP"
 		(at 27.94 158.75 90)
 		(effects
@@
 		)
 	)
+	(symbol
+		(lib_id "Jumper:SolderJumper_2_Bridged")
+		(at 124.46 165.1 0)
+		(unit 1)
+		(exclude_from_sim no)
+		(in_bom no)
+		(on_board yes)
+		(dnp no)
+		(property "Reference" "SJ1"
+			(at 124.46 163.068 0)
+			(show_name no)
+			(do_not_autoplace no)
+			(effects
+				(font
+					(size 1.27 1.27)
+				)
+			)
+		)
+		(property "Value" "DRY (cut)"
+			(at 124.46 167.64 0)
+			(show_name no)
+			(do_not_autoplace no)
+			(effects
+				(font
+					(size 1.27 1.27)
+				)
+			)
+		)
+		(property "Footprint" "Jumper:SolderJumper-2_P1.3mm_Bridged_RoundedPad1.0x1.5mm"
+			(at 124.46 165.1 0)
+			(show_name no)
+			(do_not_autoplace no)
+			(hide yes)
+			(effects
+				(font
+					(size 1.27 1.27)
+				)
+			)
+		)
+		(property "Datasheet" ""
+			(at 124.46 171.45 0)
+			(show_name no)
+			(do_not_autoplace no)
+			(hide yes)
+			(effects
+				(font
+					(size 1.27 1.27)
+				)
+			)
+		)
+		(property "Description" "Solder Jumper, 2-pole, closed/bridged"
+			(at 124.46 170.18 0)
+			(show_name no)
+			(do_not_autoplace no)
+			(hide yes)
+			(effects
+				(font
+					(size 1.27 1.27)
+				)
+			)
+		)
+		(property "ki_keywords" "solder jumper SPST"
+			(at 124.46 165.1 0)
+			(show_name no)
+			(do_not_autoplace no)
+			(hide yes)
+			(effects
+				(font
+					(size 1.27 1.27)
+				)
+			)
+		)
+		(property "ki_fp_filters" "SolderJumper*Bridged*"
+			(at 124.46 165.1 0)
+			(show_name no)
+			(do_not_autoplace no)
+			(hide yes)
+			(effects
+				(font
+					(size 1.27 1.27)
+				)
+			)
+		)
+		(property "Note" "Bridged by default. Cut it (and remove the fuse) to make COM/NO/NC a dry contact."
+			(at 124.46 165.1 0)
+			(effects
+				(font
+					(size 1.27 1.27)
+				)
+				(hide yes)
+			)
+		)
+		(pin "1"
+		)
+		(pin "2"
+		)
+		(instances
+			(project "VanController"
+				(path "/a40173d8-9ce3-58d6-b907-2ebe6d892436/c3797fdd-53b5-5939-903b-7d05619c6858/bc0adf80-6c07-5b36-899e-45ebacd85a9f"
+					(reference "SJ1")
+					(unit 1)
+				)
+				(path "/a40173d8-9ce3-58d6-b907-2ebe6d892436/c3797fdd-53b5-5939-903b-7d05619c6858/bf1ec584-e2c9-53f6-b25e-af77af5a92a6"
+					(reference "SJ2")
+					(unit 1)
+				)
+				(path "/a40173d8-9ce3-58d6-b907-2ebe6d892436/c3797fdd-53b5-5939-903b-7d05619c6858/b9c8393e-5ab4-5dc6-b8e5-ec4d7e220de4"
+					(reference "SJ3")
+					(unit 1)
+				)
+				(path "/a40173d8-9ce3-58d6-b907-2ebe6d892436/c3797fdd-53b5-5939-903b-7d05619c6858/825474ea-4786-557f-a724-6f91812a3181"
+					(reference "SJ4")
+					(unit 1)
+				)
+				(path "/a40173d8-9ce3-58d6-b907-2ebe6d892436/c3797fdd-53b5-5939-903b-7d05619c6858/ec205e71-2bbe-548f-b2eb-59f628cace52"
+					(reference "SJ5")
+					(unit 1)
+				)
+				(path "/a40173d8-9ce3-58d6-b907-2ebe6d892436/c3797fdd-53b5-5939-903b-7d05619c6858/03ce8bd4-3f6d-5c15-a6a6-cf05f7ea06f3"
+					(reference "SJ6")
+					(unit 1)
+				)
+			)
+		)
+	)
+	(wire
+		(pts
+			(xy 119.38 165.1)
+			(xy 116.84 165.1)
+		)
+		(stroke
+			(width 0)
+			(type default)
+		)
+	)
+	(label "OUT_F"
+		(at 116.84 165.1 180)
+		(effects
+			(font
+				(size 1.27 1.27)
+			)
+			(justify right bottom)
+		)
+	)
+	(wire
+		(pts
+			(xy 129.54 165.1)
+			(xy 132.08 165.1)
+		)
+		(stroke
+			(width 0)
+			(type default)
+		)
+	)
+	(label "SENSE_TAP"
+		(at 132.08 165.1 0)
+		(effects
+			(font
+				(size 1.27 1.27)
+			)
+			(justify left bottom)
+		)
+	)
